File: PTP_Darijo_Matesic_Project1/PTP_Darijo_Matesic_Project1.kicad_pcb (KiCad board)
At the start: 2 copper layers, 45 parts, among them J1 Screw_Terminal_01x02, SW1 SW_Push, SW2 SW_Wuerth_450301014042, U1 LM2574N-5, U2 NE555P, U3 SN74LVC1G11, U4 4027, U5 4027, U6 74LS47, U7 FYS-3911BUHR-21

Commit message: gt
t
Parts:
- R1, R2, R3, R4: footprint Resistor_THT:R_Axial_DIN0207_L6.3mm_D2.5mm_P10.16mm_Horizontal -> Resistor_SMD:R_1206_3216Metric_Pad1.30x1.75mm_HandSolder
- R5, R6, R7, R8: footprint Resistor_SMD:R_1206_3216Metric_Pad1.30x1.75mm_HandSolder -> Resistor_THT:R_Axial_DIN0207_L6.3mm_D2.5mm_P10.16mm_Horizontal
- moved H2 205.5 mm to (183.5, 93.0)
- moved H3 205.1 mm to (184.0, 28.5)
- moved C1 148.8 mm to (103.5, 31.2)
- moved R12 141.5 mm to (138.0, 78.5), turned to 90 degrees
- moved C2 139.0 mm to (123.0, 31.7)
- moved U1 139.0 mm to (111.2, 38.5)
- moved L1 132.5 mm to (128.0, 43.7), turned to 90 degrees
- moved J1 128.7 mm to (96.1, 47.5)
- moved R9 123.8 mm to (100.9, 75.5)
- moved R11 108.2 mm to (132.0, 78.5), turned to 90 degrees
- moved U7 100.3 mm to (165.5, 55.0)
- moved R13 99.1 mm to (135.0, 78.5), turned to 90 degrees
- moved C4 97.3 mm to (80.5, 49.5)
- moved H4 96.0 mm to (77.5, 93.5)
- moved R10 95.7 mm to (129.0, 78.5), turned to 90 degrees
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Routing:
- net +5V: track 0.00 -> 287.1 mm
- net GND: track 0.00 -> 103.5 mm
- net CLOCK: track 0.00 -> 40.6 mm
- net Net-(D1-K): track 0.00 -> 38.2 mm
- net Net-(U7-C): track 0.00 -> 37.7 mm
- net VDD: track 0.00 -> 33.3 mm
- net Net-(U2-THR): track 0.00 -> 32.0 mm
- net RESET: track 0.00 -> 28.4 mm
- net Net-(U4A-J): track 0.00 -> 22.4 mm
- net Net-(SW2-A): track 0.00 -> 22.3 mm
- net Net-(U7-A): track 0.00 -> 19.5 mm
- net Net-(U4B-J): track 0.00 -> 17.5 mm
- net Net-(U2-DIS): track 0.00 -> 17.1 mm
- net Net-(U5A-J): track 0.00 -> 16.8 mm
- net Net-(U7-E): track 0.00 -> 15.1 mm
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
Commit message: a
a
Parts:
- moved H2 21.2 mm to (169.0, 77.5)
- moved H4 16.8 mm to (82.5, 77.5)
- moved H3 15.0 mm to (169.0, 28.5)
- moved C4 9.91 mm to (90.0, 52.5)
- moved R4 9.91 mm to (89.5, 57.0)
- moved SW1 9.91 mm to (78.7, 52.2)
- moved R5 6.06 mm to (158.9, 37.6)
- moved R6 5.49 mm to (151.5, 37.6)
- moved R7 5.49 mm to (144.0, 37.6)
- moved R8 5.44 mm to (136.5, 37.5)
- moved R1 5.15 mm to (86.9, 65.0)
- moved R2 5.15 mm to (86.9, 61.0)
- moved H1 5.02 mm to (82.5, 28.5)
- moved D2 4.59 mm to (159.4, 42.0)
- moved D3 4.59 mm to (151.9, 42.0)
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Routing:
- net +5V: track 287.1 -> 139.5 mm
- net Q1: track 0.00 -> 78.0 mm, vias 0 -> 1
- net Q0: track 10.8 -> 82.0 mm
- net Q3: track 0.00 -> 61.0 mm, vias 0 -> 1
- net Net-(U7-B): track 0.77 -> 32.2 mm
- net Q2: track 2.04 -> 32.9 mm, vias 0 -> 1
- net Net-(U6-BI): track 0.00 -> 25.5 mm
- net GND: track 103.5 -> 123.2 mm, vias 0 -> 1
- net Net-(U2-THR): track 32.0 -> 50.6 mm
- net Net-(D1-K): track 38.2 -> 50.1 mm
- net Net-(SW2-A): track 22.3 -> 11.9 mm
- net CLOCK: track 40.6 -> 49.4 mm
- net Net-(U7-C): track 37.7 -> 29.1 mm
- net Net-(U5B-J): track 14.3 -> 21.6 mm
- net Net-(U7-D): track 9.47 -> 16.0 mm
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